File: SiboorVoronExt/SiboorVoronExt.kicad_pcb (KiCad board)
At the start: 2 copper layers, 40.7 x 29.8 mm, 45 parts, among them Q1 BSS138, U1 74LVC1G17, U2 74LVC1G17, U3 MP1584EN, U4 AMS1117-3.3

Commit message: Frist PCB Draft
Parts:
- U1, U2: footprint Package_TO_SOT_SMD:SOT-23-5_HandSoldering -> SMD:SOT-23-5_HandSoldering
- U4: footprint Package_TO_SOT_SMD:SOT-223-3_TabPin2 -> SMD:SOT-223-3_TabPin2
- moved D5 144.4 mm to (5.10, 9.00), turned to 180 degrees
- moved R15 139.8 mm to (8.44, 9.00), turned to 180 degrees
- moved D6 138.9 mm to (5.08, 18.0), turned to 180 degrees
- moved R13 138.1 mm to (15.3, 13.8), turned to 90 degrees
- moved R11 135.8 mm to (20.1, 22.0)
- moved C9 135.4 mm to (1.56, 7.95), turned to 90 degrees
- moved R16 134.5 mm to (7.90, 18.9), turned to 90 degrees
- moved U2 134.1 mm to (4.40, 20.9)
- moved R10 134.0 mm to (0.95, 21.1)
- moved FAN1 133.6 mm to (14.8, 25.7)
- moved RGB2 133.6 mm to (3.89, 25.7)
- moved TH1 133.6 mm to (23.3, 25.6)
- moved RGB1 133.6 mm to (31.7, 25.7)
- moved D3 133.6 mm to (16.2, 22.1)
- moved U4 133.5 mm to (5.30, 13.6)
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Routing:
- net +5V: track 0.00 -> 81.7 mm
- net +24V: track 0.00 -> 60.2 mm, vias 0 -> 4
- net TH: track 0.00 -> 49.1 mm, vias 0 -> 1
- net FAN_PWM: track 0.00 -> 36.4 mm
- net +3.3V: track 0.00 -> 34.1 mm, vias 0 -> 2
- net RGB2: track 0.00 -> 25.7 mm, vias 0 -> 1
- net RGB1: track 0.00 -> 25.1 mm
- net Net-(D1-A): track 0.00 -> 19.2 mm
- net Net-(U3-FB): track 0.00 -> 17.5 mm, vias 0 -> 2
- net Net-(D2-K): track 0.00 -> 15.9 mm
- net VDD: track 0.00 -> 14.5 mm, vias 0 -> 6
- net Net-(TH1-Pin_1): track 0.00 -> 11.4 mm
- net Net-(D3-K): track 0.00 -> 11.1 mm
- net Net-(RGB1-Pin_2): track 0.00 -> 6.36 mm
- net Net-(U3-COMP): track 0.00 -> 5.19 mm
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Other:
- board size 40.7 x 29.8 mm -> 40.6 x 30 mm

Commit message: V1.0
Parts:
- Q1: footprint Package_TO_SOT_SMD:SOT-23_Handsoldering -> SMD:SOT-23_Handsoldering
- U3: footprint Package_SO:SOIC-8-1EP_3.9x4.9mm_P1.27mm_EP2.29x3mm_ThermalVias -> SMD:SOIC-8-1EP_3.9x4.9mm_P1.27mm_EP2.29x3mm_ThermalVias
- moved EXT1 10.5 mm to (5.05, 5.90), turned to 90 degrees
- moved EXT2 10.5 mm to (25.6, 5.88), turned to 90 degrees
- moved 24V1 0.19 mm to (36.8, 15.0)
- moved Q1 0.18 mm to (11.5, 21.0)
- moved C1 0.09 mm to (25.9, 21.1)
- moved C2 0.08 mm to (27.8, 20.8)
- moved C4 0.08 mm to (29.8, 21.1)
- moved R5 0.07 mm to (31.3, 21.1)
- moved C6 0.06 mm to (33.0, 15.5)
- moved R3 0.06 mm to (30.8, 18.2)
- moved R4 0.06 mm to (27.3, 18.2)
Connections:
- 24V1 pad 1: GND -> +24V
- 24V1 pad 2: +24V -> GND
Routing:
- net +5V: track 81.7 -> 110.4 mm, vias 0 -> 2
- net FAN_PWM: track 36.4 -> 26.3 mm
- net VDD: track 14.5 -> 20.2 mm
- net TH: track 49.1 -> 44.1 mm
- net RGB1: track 25.1 -> 27.3 mm
- net +24V: track 60.2 -> 58.3 mm
- net Net-(D5-K): track 0.00 -> 1.55 mm
- net Net-(D3-K): track 11.1 -> 10.3 mm
- net GND: vias 0 -> 48
- added copper zone on B.Cu, net GND
- added copper zone on F.Cu, net GND
Other:
- board text added: "+"
- board text added: "-"
- board text added: "24V"
- board text added: "EXP1"
- board text added: "EXP2"
- board text added: "FAN"
- board text added: "RGB1"
- board text added: "RGB2"
- board text added: "S"
- board text added: "SIBOOR GEMINI V3 EXTENSION BOARD"
- board text added: "TH"

Commit message: up
Parts:
- removed JP1: SolderJumper_2_Open, Jumper:SolderJumper-2_P1.3mm_Open_RoundedPad1.0x1.5mm
- C2, C7: value 10u/25V/0805 -> 10u/25V/1206; footprint Capacitor_SMD:C_0805_2012Metric_Pad1.18x1.45mm_HandSolder -> SMD:C_1206_HandSolder
- C5, C6: value 10u/25V/0805 -> 10u/25V/1206; footprint Capacitor_SMD:C_0805_2012Metric_Pad1.18x1.45mm_HandSolder -> Capacitor_SMD:C_1206_3216Metric_Pad1.33x1.80mm_HandSolder
- C8: value 10u/25V/0805 -> 10u/25V/1206; footprint Capacitor_SMD:C_0805_2012Metric_Pad1.18x1.45mm_HandSolder -> Resistor_SMD:R_0805_2012Metric_Pad1.20x1.40mm_HandSolder
- D1: footprint Diode_SMD:D_SOD-323 -> Diode_SMD:D_SOD-123
- D2: footprint Diode_SMD:D_SMB_Handsoldering -> myLib_SMD:D_SMB_Handsoldering
- L2: footprint Inductor_SMD:L_Wuerth_WE-PD2-Typ-L -> SMD:L_8.0x7.5
- R6, R7: footprint Resistor_SMD:R_0603_1608Metric_Pad0.98x0.95mm_HandSolder -> Resistor_SMD:R_0805_2012Metric_Pad1.20x1.40mm_HandSolder
- moved EXP2 10.5 mm to (35.7, 3.30), turned to -90 degrees
- moved EXP1 10.4 mm to (15.2, 3.33), turned to -90 degrees
- moved C1 1.74 mm to (27.0, 19.7), turned to 180 degrees
- moved C4 1.22 mm to (31.0, 21.1)
- moved R5 1.20 mm to (32.5, 21.1)
- moved R13 1.18 mm to (14.4, 14.5), turned to 0 degrees
- moved C8 0.92 mm to (15.0, 11.0)
- moved C5 0.84 mm to (32.8, 10.9)
- moved R2 0.82 mm to (29.9, 9.05)
- moved C3 0.78 mm to (26.5, 9.05)
- moved R3 0.78 mm to (30.0, 18.1)
- moved R6 0.78 mm to (20.3, 4.70)
- moved C2 0.76 mm to (27.7, 21.6), turned to 0 degrees
- moved C7 0.74 mm to (12.7, 10.8)
- moved R4 0.62 mm to (26.7, 18.1)
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- renumbered EXT1 to EXP1, EXT2 to EXP2
Connections:
- EXP1 pad 10: VDD -> +5V
- RGB1 pad 1: +5V -> Net-(RGB1-Pin_1)
- RGB1 pad 2: Net-(RGB1-Pin_2) -> +5V
- RGB2 pad 1: +5V -> Net-(RGB2-Pin_1)
- RGB2 pad 2: Net-(RGB2-Pin_2) -> +5V
- U1 pad 4: Net-(RGB1-Pin_2) -> Net-(RGB1-Pin_1)
- U2 pad 4: Net-(RGB2-Pin_2) -> Net-(RGB2-Pin_1)
- U4 pad 3: VDD -> +5V
Routing:
- net VDD: track 20.2 -> 0.00 mm, vias 6 -> 0
- net +5V: track 110.4 -> 122.4 mm, vias 2 -> 9
- net FAN_PWM: track 26.3 -> 37.7 mm
- net Net-(RGB1-Pin_1): track 0.00 -> 8.65 mm
- net Net-(RGB1-Pin_2): track 6.36 -> 0.00 mm
- net Net-(RGB2-Pin_1): track 0.00 -> 5.20 mm
- net TH: track 44.1 -> 49.1 mm
- net Net-(RGB2-Pin_2): track 3.99 -> 0.00 mm
- net Net-(D2-K): track 15.9 -> 18.5 mm
- net +24V: track 58.3 -> 60.8 mm
- net RGB1: track 27.3 -> 25.1 mm
- net Net-(D3-K): track 10.3 -> 8.53 mm
- net Net-(D1-A): track 19.2 -> 18.6 mm
- net Net-(U3-EN): track 3.90 -> 3.35 mm
- net GND: vias 48 -> 49
