File: SiboorVoronExt/SiboorVoronExt.kicad_sch (KiCad schematic)
At the start: 4 parts, among them J1 Conn_02x05_Odd_Even, J2 Conn_02x05_Odd_Even, U1 74LVC1G17, U2 74LVC1G17

Commit message: First Placement
Parts:
- added 24V1, FAN1, TH1: Conn_01x02, Connector_JST:JST_XH_B2B-XH-A_1x02_P2.50mm_Vertical, symbol Connector_Generic:Conn_01x02
- added C1, C3: 100n/50V/0603, Capacitor_SMD:C_0603_1608Metric_Pad1.08x0.95mm_HandSolder, symbol Device:C_Small
- added C2, C5, C6, C7, C8, C9: 10u/25V/0805, Capacitor_SMD:C_0805_2012Metric_Pad1.18x1.45mm_HandSolder, symbol Device:C_Small
- added C4: 150p/50V/0603, Capacitor_SMD:C_0603_1608Metric_Pad1.08x0.95mm_HandSolder, symbol Device:C_Small
- added D1: 1N5819WS, Diode_SMD:D_SOD-323, symbol Device:D_Schottky_Small
- added D2: SS34/SMB, Diode_SMD:D_SMB_Handsoldering, symbol Device:D_Schottky_Small
- added D3, D4, D5, D6: Red/20mA/0603, LED_SMD:LED_0603_1608Metric_Pad1.05x0.95mm_HandSolder, symbol Device:LED_Small
- added JP1: SolderJumper_2_Open, Jumper:SolderJumper-2_P1.3mm_Open_RoundedPad1.0x1.5mm, symbol Jumper:SolderJumper_2_Open
- added L2: 15uH/3A, Inductor_SMD:L_Wuerth_WE-PD2-Typ-L, symbol Device:L_Small
- added Q1: BSS138, Package_TO_SOT_SMD:SOT-23_Handsoldering, symbol Device:Q_NMOS_GSD
- added R1: 1k/0603, Resistor_SMD:R_0603_1608Metric_Pad0.98x0.95mm_HandSolder, symbol Device:R_Small
- added R10, R9: 10k/0603, Resistor_SMD:R_0603_1608Metric_Pad0.98x0.95mm_HandSolder, symbol Device:R_Small
- added R11: 4k7/0.1%/0603, Resistor_SMD:R_0603_1608Metric_Pad0.98x0.95mm_HandSolder, symbol Device:R_Small
- added R12: 100R/0603, Resistor_SMD:R_0603_1608Metric_Pad0.98x0.95mm_HandSolder, symbol Device:R_Small
- added R13, R14: 22k, Resistor_SMD:R_0603_1608Metric_Pad0.98x0.95mm_HandSolder, symbol Device:R_Small
- added R15: 1k, Resistor_SMD:R_0603_1608Metric_Pad0.98x0.95mm_HandSolder, symbol Device:R_Small
- added R16: 560R, Resistor_SMD:R_0603_1608Metric_Pad0.98x0.95mm_HandSolder, symbol Device:R_Small
- added R2, R3, R5, R8: 100k/0603, Resistor_SMD:R_0603_1608Metric_Pad0.98x0.95mm_HandSolder, symbol Device:R_Small
- added R4: 24.9k/0603, Resistor_SMD:R_0603_1608Metric_Pad0.98x0.95mm_HandSolder, symbol Device:R_Small
- added R6: 40.2k/0603, Resistor_SMD:R_0603_1608Metric_Pad0.98x0.95mm_HandSolder, symbol Device:R_Small
- added R7: 210k/0603, Resistor_SMD:R_0603_1608Metric_Pad0.98x0.95mm_HandSolder, symbol Device:R_Small
- added RGB1, RGB2: Conn_01x03, Connector_JST:JST_XH_B3B-XH-A_1x03_P2.50mm_Vertical, symbol Connector_Generic:Conn_01x03
- added U3: MP1584EN, Package_SO:SOIC-8-1EP_3.9x4.9mm_P1.27mm_EP2.29x3mm_ThermalVias, symbol Olimex_IC:MP1584EN(SOIC8E)
- added U4: AMS1117-3.3, Package_TO_SOT_SMD:SOT-223-3_TabPin2, symbol Regulator_Linear:AMS1117-3.3
- EXT1: renamed from J1; footprint (none) -> Connector_PinHeader_2.54mm:PinHeader_2x05_P2.54mm_Vertical
- EXT2: renamed from J2; footprint (none) -> Connector_PinHeader_2.54mm:PinHeader_2x05_P2.54mm_Vertical
- U1, U2: footprint (none) -> Package_TO_SOT_SMD:SOT-23-5_HandSoldering
Connections:
- net RGB1: now reaches U1.2
- net RGB1: now also EXT2.6 (Pin_6), R9.2
- net GND: now reaches U1.3 (GND)
- net GND: now also EXT1.9 (Pin_9), EXT2.9 (Pin_9), U2.3 (GND), 24V1.1 (Pin_1), C1.1, C2.2, C5.2, C6.2, C7.2, C8.2, C9.2, D2.2 (A), Q1.2 (S), R10.1, R14.1, R15.1, R16.1, R2.1, R4.1, R5.1, R6.1, R8.1, R9.1, RGB1.3 (Pin_3), RGB2.3 (Pin_3), TH1.2 (Pin_2), U3.5 (GND), U3.9 (EP), U4.1 (GND)
- net at U1.4: now also RGB1.2 (Pin_2)
- net +5V: now reaches U1.5 (VCC)
- net +5V: now also U2.5 (VCC), C7.1, C8.1, D5.2 (A), JP1.1 (A), L2.2, R7.2, RGB1.1 (Pin_1), RGB2.1 (Pin_1)
- net FAN_PWM: now reaches EXT2.1 (Pin_1)
- net FAN_PWM: now also R12.1
- net TH: now reaches EXT2.7 (Pin_7)
- net TH: now also R1.1
- net VDD: now reaches EXT1.10 (Pin_10)
- net VDD: now also JP1.2 (B), U4.3 (VI)
- net RGB2: now reaches EXT1.5 (Pin_5)
- net RGB2: now also U2.2, R10.2
- net at U2.4: now also RGB2.2 (Pin_2)
- new net: Q1.1 (G), R12.2, R8.2
- new net: D1.2 (A), FAN1.2 (Pin_2), Q1.3 (D), R13.1
- new net: C1.2, C2.1, R1.2, R11.1, TH1.1 (Pin_1)
- new net: R6.2, R7.1, U3.4 (FB)
- new net: D5.1 (K), R15.2
- new net: D6.1 (K), R16.2
- new net: C4.2, R5.2
- new net: D3.1 (K), R13.2
- new net: R3.1, R4.2, U3.2 (EN)
- new net: C3.2, D2.1 (K), L2.1, U3.1 (SW)
- new net: C4.1, U3.3 (COMP)
- new net: R2.2, U3.6 (FREQ)
- new net: C3.1, U3.8 (BST)
- new net: D4.1 (K), R14.2
- new net +24V: 24V1.2 (Pin_2), C5.1, C6.1, D1.1 (K), D3.2 (A), D4.2 (A), FAN1.1 (Pin_1), R3.2, U3.7 (VIN)
- new net +3.3V: C9.1, D6.2 (A), R11.2, U4.2 (VO)
Other:
- moved on the sheet: EXT1, EXT2, U1, U2

Commit message: V1.0
Parts:
- Q1: footprint Package_TO_SOT_SMD:SOT-23_Handsoldering -> SMD:SOT-23_Handsoldering
- U1, U2: footprint Package_TO_SOT_SMD:SOT-23-5_HandSoldering -> SMD:SOT-23-5_HandSoldering
- U3: footprint Package_SO:SOIC-8-1EP_3.9x4.9mm_P1.27mm_EP2.29x3mm_ThermalVias -> SMD:SOIC-8-1EP_3.9x4.9mm_P1.27mm_EP2.29x3mm_ThermalVias
- U4: footprint Package_TO_SOT_SMD:SOT-223-3_TabPin2 -> SMD:SOT-223-3_TabPin2
Connections:
- net +24V: now also 24V1.1 (Pin_1); no longer 24V1.2 (Pin_2)
- net GND: now also 24V1.2 (Pin_2); no longer 24V1.1 (Pin_1)
Changed lines of the file:
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@@
     (stroke (width 0) (type default))
   )
-  (wire (pts (xy 29.21 116.84) (xy 33.02 116.84))
+  (wire (pts (xy 30.48 116.84) (xy 33.02 116.84))
     (stroke (width 0) (type default))
   )
@@
     (stroke (width 0) (type default))
   )
-  (wire (pts (xy 29.21 114.3) (xy 33.02 114.3))
+  (wire (pts (xy 30.48 114.3) (xy 33.02 114.3))
     (stroke (width 0) (type default))
   )
@@
       (effects (font (size 1.27 1.27)) (justify left))
     )
-    (property "Footprint" "Package_TO_SOT_SMD:SOT-23_Handsoldering" (at 64.77 52.07 0)
+    (property "Footprint" "SMD:SOT-23_Handsoldering" (at 64.77 52.07 0)
       (effects (font (size 1.27 1.27)) hide)
     )
@@
     )
   )
-  (symbol (lib_id "Connector_Generic:Conn_01x02") (at 24.13 116.84 180) (unit 1)
-    (in_bom yes) (on_board yes) (dnp no) (fields_autoplaced)
-    (property "Reference" "24V1" (at 24.13 109.22 0)
-      (effects (font (size 1.27 1.27)))
-    )
-    (property "Value" "Conn_01x02" (at 24.13 111.76 0)
-      (effects (font (size 1.27 1.27)))
-    )
-    (property "Footprint" "Connector_JST:JST_XH_B2B-XH-A_1x02_P2.50mm_Vertical" (at 24.13 116.84 0)
-      (effects (font (size 1.27 1.27)) hide)
-    )
-    (property "Datasheet" "~" (at 24.13 116.84 0)
-      (effects (font (size 1.27 1.27)) hide)
-    )
-    (pin "1")
-    (pin "2")
-    (instances
-      (project "SiboorVoronExt"
-        (path "/1531a0b2-1993-44d2-b6f7-c211d58ab3cb"
-          (reference "24V1") (unit 1)
-        )
-      )
-    )
-  )
   (symbol (lib_id "Device:R_Small") (at 107.95 177.8 180) (unit 1)
     (in_bom yes) (on_board yes) (dnp no)
@@
       (effects (font (size 1.27 1.27)))
     )
-    (property "Footprint" "Package_TO_SOT_SMD:SOT-23-5_HandSoldering" (at 214.63 46.99 0)
+    (property "Footprint" "SMD:SOT-23-5_HandSoldering" (at 214.63 46.99 0)
       (effects (font (size 1.27 1.27)) hide)
     )
@@
         (path "/1531a0b2-1993-44d2-b6f7-c211d58ab3cb"
           (reference "D5") (unit 1)
+        )
+      )
+    )
+  )
+  (symbol (lib_id "Connector_Generic:Conn_01x02") (at 25.4 114.3 0) (mirror y) (unit 1)
+    (in_bom yes) (on_board yes) (dnp no)
+    (property "Reference" "24V1" (at 25.4 121.92 0)
+      (effects (font (size 1.27 1.27)))
+    )
+    (property "Value" "Conn_01x02" (at 25.4 119.38 0)
+      (effects (font (size 1.27 1.27)))
+    )
+    (property "Footprint" "Connector_JST:JST_XH_B2B-XH-A_1x02_P2.50mm_Vertical" (at 25.4 114.3 0)
+      (effects (font (size 1.27 1.27)) hide)
+    )
+    (property "Datasheet" "~" (at 25.4 114.3 0)
+      (effects (font (size 1.27 1.27)) hide)
+    )
+    (pin "1")
+    (pin "2")
+    (instances
+      (project "SiboorVoronExt"
+        (path "/1531a0b2-1993-44d2-b6f7-c211d58ab3cb"
+          (reference "24V1") (unit 1)
         )
       )
@@
       (effects (font (size 1.524 1.524)))
     )
-    (property "Footprint" "Package_SO:SOIC-8-1EP_3.9x4.9mm_P1.27mm_EP2.29x3mm_ThermalVias" (at 68.58 160.02 0)
+    (property "Footprint" "SMD:SOIC-8-1EP_3.9x4.9mm_P1.27mm_EP2.29x3mm_ThermalVias" (at 68.58 160.02 0)
       (effects (font (size 1.27 1.27)) hide)
     )
@@
       (effects (font (size 1.27 1.27)))
     )
-    (property "Footprint" "Package_TO_SOT_SMD:SOT-23-5_HandSoldering" (at 214.63 71.12 0)
+    (property "Footprint" "SMD:SOT-23-5_HandSoldering" (at 214.63 71.12 0)
       (effects (font (size 1.27 1.27)) hide)
     )
@@
       (effects (font (size 1.27 1.27)))
     )
-    (property "Footprint" "Package_TO_SOT_SMD:SOT-223-3_TabPin2" (at 157.48 154.94 0)
-      (effects (font (size 1.27 1.27)) hide)
-    )
+    (property "Footprint" "SMD:SOT-223-3_TabPin2" (at 157.48 154.94 0)
+      (effects (font (size 1.27 1.27)) hide)
+    )

Commit message: up
Parts:
- removed JP1: SolderJumper_2_Open, Jumper:SolderJumper-2_P1.3mm_Open_RoundedPad1.0x1.5mm, symbol Jumper:SolderJumper_2_Open
- C2, C7: value 10u/25V/0805 -> 10u/25V/1206; footprint Capacitor_SMD:C_0805_2012Metric_Pad1.18x1.45mm_HandSolder -> SMD:C_1206_HandSolder
- C5, C6: value 10u/25V/0805 -> 10u/25V/1206; footprint Capacitor_SMD:C_0805_2012Metric_Pad1.18x1.45mm_HandSolder -> Capacitor_SMD:C_1206_3216Metric_Pad1.33x1.80mm_HandSolder
- C8: value 10u/25V/0805 -> 10u/25V/1206; footprint Capacitor_SMD:C_0805_2012Metric_Pad1.18x1.45mm_HandSolder -> Resistor_SMD:R_0805_2012Metric_Pad1.20x1.40mm_HandSolder
- D1: footprint Diode_SMD:D_SOD-323 -> Diode_SMD:D_SOD-123
- D2: footprint Diode_SMD:D_SMB_Handsoldering -> myLib_SMD:D_SMB_Handsoldering
- L2: footprint Inductor_SMD:L_Wuerth_WE-PD2-Typ-L -> SMD:L_8.0x7.5
- R6, R7: footprint Resistor_SMD:R_0603_1608Metric_Pad0.98x0.95mm_HandSolder -> Resistor_SMD:R_0805_2012Metric_Pad1.20x1.40mm_HandSolder
- renumbered EXT1 to EXP1, EXT2 to EXP2
Connections:
- net VDD is gone; now on net +5V: EXP1.10 (Pin_10), U4.3 (VI)
- net +5V: now also RGB1.2 (Pin_2), RGB2.2 (Pin_2); no longer RGB1.1 (Pin_1), RGB2.1 (Pin_1)
- net at U1.4: now also RGB1.1 (Pin_1); no longer RGB1.2 (Pin_2)
- net at U2.4: now also RGB2.1 (Pin_1); no longer RGB2.2 (Pin_2)
Other:
- moved on the sheet: RGB1, RGB2
